File: ov-twin.kicad_pcb (KiCad board)
At the start: 4 copper layers, 64 x 64 mm, 31 parts, among them J1 USB_C_Receptacle_USB2.0, J3 Conn_01x02, U1 NCP1117-3.3_SOT223, U2 RP2040, U4 W25Q128JVS, Y1 Crystal_GND24

Commit message: Hub and stuff
Parts:
- added C17: 27p, Capacitor_SMD:C_0402_1005Metric, F.Cu at (179.0, 102.0)
- added C19: 27p, Capacitor_SMD:C_0402_1005Metric, F.Cu at (183.8, 102.0)
- added C20: 1u, Capacitor_SMD:C_0402_1005Metric, F.Cu at (189.4, 90.0)
- added C21: 1u, Capacitor_SMD:C_0402_1005Metric, F.Cu at (184.8, 100.0)
- added C22: 1u, Capacitor_SMD:C_0402_1005Metric, F.Cu at (179.0, 92.0)
- added C23: 1u, Capacitor_SMD:C_0402_1005Metric, F.Cu at (184.4, 88.5)
- added C24: 1u, Capacitor_SMD:C_0402_1005Metric, F.Cu at (189.4, 91.0)
- added C25: 1u, Capacitor_SMD:C_0402_1005Metric, F.Cu at (189.4, 92.0)
- added C26: 1u, Capacitor_SMD:C_0402_1005Metric, F.Cu at (189.4, 95.6)
- added C27: 1u, Capacitor_SMD:C_0402_1005Metric, F.Cu at (179.0, 95.6)
- added C28: 1u, Capacitor_SMD:C_0402_1005Metric, F.Cu at (185.4, 88.5)
- added C29: 1u, Capacitor_SMD:C_0402_1005Metric, F.Cu at (183.4, 88.5)
- added C30: 1u, Capacitor_SMD:C_0402_1005Metric, F.Cu at (186.4, 88.5)
- added C31: 1u, Capacitor_SMD:C_0805_2012Metric, F.Cu at (179.8, 82.5)
- added C32: 1u, Capacitor_SMD:C_0402_1005Metric, F.Cu at (185.8, 100.0)
- added J2: Conn_01x02, Connector_PinHeader_2.54mm:PinHeader_1x02_P2.54mm_Vertical, F.Cu at (216.7, 86.0)
- added R11: 1k, Resistor_SMD:R_0402_1005Metric, F.Cu at (177.0, 83.0)
- added R12: DNF, Resistor_SMD:R_0402_1005Metric, F.Cu at (175.0, 83.0)
- added R13: 1k, Resistor_SMD:R_0402_1005Metric, F.Cu at (183.8, 100.0)
- added R14: 10k, Resistor_SMD:R_0402_1005Metric, F.Cu at (186.8, 100.0)
- added R7: 27, Resistor_SMD:R_0402_1005Metric, F.Cu at (188.4, 86.3)
- added R8: 27, Resistor_SMD:R_0402_1005Metric, F.Cu at (187.4, 86.3)
- added U3: RP2040, ov-twin:RP2040-QFN-56, F.Cu at (184.2, 94.6)
- added U5: W25Q128JVS, Package_SO:SOIC-8_5.23x5.23mm_P1.27mm, F.Cu at (178.1, 86.5)
- added Y2: Crystal_GND24, Crystal:Crystal_SMD_3225-4Pin_3.2x2.5mm, F.Cu at (181.4, 102.0)
- moved C18 78.4 mm to (159.8, 82.5)
- moved J1 77.5 mm to (172.0, 62.3), turned to 180 degrees
- moved U2 13.5 mm to (164.2, 94.6)
- moved C1 13.5 mm to (169.4, 90.0)
- moved C10 13.5 mm to (166.4, 88.5)
- moved C11 13.5 mm to (163.4, 88.5)
- moved C12 13.5 mm to (165.8, 100.0)
- moved C15 13.5 mm to (159.0, 102.0)
- moved C16 13.5 mm to (163.8, 102.0)
- moved C2 13.5 mm to (169.4, 91.0)
- moved C3 13.5 mm to (165.4, 88.5)
- moved C4 13.5 mm to (164.4, 88.5)
- moved C5 13.5 mm to (169.4, 95.6)
- moved C6 13.5 mm to (169.4, 92.0)
- moved C7 13.5 mm to (164.8, 100.0)
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Routing:
- net /pi-b-qspi-ss: track 0.00 -> 16.7 mm, vias 0 -> 2
- net /pi-b-qspi-sd2: track 0.00 -> 12.5 mm, vias 0 -> 2
- net GND: track 12.3 -> 24.6 mm, vias 7 -> 14
- net /pi-b-qspi-sd1: track 0.00 -> 11.0 mm, vias 0 -> 2
- net +3V3: track 10.7 -> 21.4 mm, vias 2 -> 4
- net /pi-b-qspi-sd3: track 0.00 -> 9.62 mm, vias 0 -> 2
- net /pi-b-qspi-sd0: track 0.00 -> 8.62 mm, vias 0 -> 2
- net /pi-b-qspi-sclk: track 0.00 -> 8.05 mm, vias 0 -> 2
- net Net-(U3-USB_DM): track 0.00 -> 7.39 mm, vias 0 -> 2
- net Net-(U3-USB_DP): track 0.00 -> 7.30 mm, vias 0 -> 2
- net Net-(U2-USB_DM): track 0.00 -> 7.24 mm, vias 0 -> 2
- net Net-(U2-USB_DP): track 0.00 -> 7.15 mm, vias 0 -> 2
- net +1V1: track 6.71 -> 13.4 mm, vias 2 -> 4
- net /pi-b-xin: track 0.00 -> 6.41 mm
- net Net-(C19-Pad1): track 0.00 -> 4.28 mm
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
Commit message: Mostly routed, wondering how to do sniffing
Parts:
- added C33: 27p, Capacitor_SMD:C_0402_1005Metric, F.Cu at (155.8, 70.2)
- added C34: 27p, Capacitor_SMD:C_0402_1005Metric, F.Cu at (154.8, 64.6)
- added C35: 10u, Capacitor_SMD:C_0805_2012Metric, F.Cu at (163.0, 62.2)
- added C36: 10u, Capacitor_SMD:C_0805_2012Metric, F.Cu at (159.4, 62.2)
- added D1: WS2812B, LED_SMD:LED_WS2812B-2020_PLCC4_2.0x2.0mm, F.Cu at (196.0, 64.8)
- added D10: WS2812B, LED_SMD:LED_WS2812B-2020_PLCC4_2.0x2.0mm, F.Cu at (180.4, 101.6)
- added D11: WS2812B, LED_SMD:LED_WS2812B-2020_PLCC4_2.0x2.0mm, F.Cu at (183.0, 110.0)
- added D12: WS2812B, LED_SMD:LED_WS2812B-2020_PLCC4_2.0x2.0mm, F.Cu at (180.4, 118.4)
- added D13: WS2812B, LED_SMD:LED_WS2812B-2020_PLCC4_2.0x2.0mm, F.Cu at (172.0, 122.0)
- added D14: WS2812B, LED_SMD:LED_WS2812B-2020_PLCC4_2.0x2.0mm, F.Cu at (163.6, 118.4)
- added D15: WS2812B, LED_SMD:LED_WS2812B-2020_PLCC4_2.0x2.0mm, F.Cu at (160.0, 110.0)
- added D16: WS2812B, LED_SMD:LED_WS2812B-2020_PLCC4_2.0x2.0mm, F.Cu at (163.6, 101.6)
- added D17: WS2812B, LED_SMD:LED_WS2812B-2020_PLCC4_2.0x2.0mm, F.Cu at (148.0, 87.2)
- added D18: WS2812B, LED_SMD:LED_WS2812B-2020_PLCC4_2.0x2.0mm, F.Cu at (148.0, 84.0)
- added D19: WS2812B, LED_SMD:LED_WS2812B-2020_PLCC4_2.0x2.0mm, F.Cu at (148.0, 80.8)
- added D2: WS2812B, LED_SMD:LED_WS2812B-2020_PLCC4_2.0x2.0mm, F.Cu at (196.0, 68.0)
- added D20: WS2812B, LED_SMD:LED_WS2812B-2020_PLCC4_2.0x2.0mm, F.Cu at (148.0, 77.6)
- added D21: WS2812B, LED_SMD:LED_WS2812B-2020_PLCC4_2.0x2.0mm, F.Cu at (148.0, 74.4)
- added D22: WS2812B, LED_SMD:LED_WS2812B-2020_PLCC4_2.0x2.0mm, F.Cu at (148.0, 71.2)
- added D23: WS2812B, LED_SMD:LED_WS2812B-2020_PLCC4_2.0x2.0mm, F.Cu at (148.0, 68.0)
- added D24: WS2812B, LED_SMD:LED_WS2812B-2020_PLCC4_2.0x2.0mm, F.Cu at (148.0, 64.8)
- added D3: WS2812B, LED_SMD:LED_WS2812B-2020_PLCC4_2.0x2.0mm, F.Cu at (196.0, 71.2)
- added D4: WS2812B, LED_SMD:LED_WS2812B-2020_PLCC4_2.0x2.0mm, F.Cu at (196.0, 74.4)
- added D5: WS2812B, LED_SMD:LED_WS2812B-2020_PLCC4_2.0x2.0mm, F.Cu at (196.0, 77.6)
- added D6: WS2812B, LED_SMD:LED_WS2812B-2020_PLCC4_2.0x2.0mm, F.Cu at (196.0, 80.8)
- added D7: WS2812B, LED_SMD:LED_WS2812B-2020_PLCC4_2.0x2.0mm, F.Cu at (196.0, 84.0)
- added D8: WS2812B, LED_SMD:LED_WS2812B-2020_PLCC4_2.0x2.0mm, F.Cu at (196.0, 87.2)
- added D9: WS2812B, LED_SMD:LED_WS2812B-2020_PLCC4_2.0x2.0mm, F.Cu at (172.0, 98.0)
- added JP1: SolderJumper_2_Open, Jumper:SolderJumper-2_P1.3mm_Open_TrianglePad1.0x1.5mm, F.Cu at (155.8, 62.4)
- added R15: 1k, Resistor_SMD:R_0402_1005Metric, F.Cu at (156.8, 64.6)
- added R16: 27, Resistor_SMD:R_0402_1005Metric, F.Cu at (164.4, 66.8)
- added R17: 27, Resistor_SMD:R_0402_1005Metric, F.Cu at (164.4, 67.8)
- added RV1: R_Potentiometer_MountingPin, Potentiometer_THT:Potentiometer_Alps_RK09K_Single_Vertical, F.Cu at (174.5, 103.0)
- added SW1: SW_SPST, ov-twin:k2-1817UQ, F.Cu at (152.0, 94.0)
- added SW2: SW_SPST, ov-twin:k2-1817UQ, F.Cu at (146.0, 100.0)
- added SW3: SW_SPST, ov-twin:k2-1817UQ, F.Cu at (158.0, 100.0)
- added SW4: SW_SPST, ov-twin:k2-1817UQ, F.Cu at (152.0, 106.0)
- added SW5: SW_SPST, ov-twin:k2-1817UQ, F.Cu at (192.0, 94.0)
- added SW6: SW_SPST, ov-twin:k2-1817UQ, F.Cu at (186.0, 100.0)
- added SW7: SW_SPST, ov-twin:k2-1817UQ, F.Cu at (198.0, 100.0)
- added SW8: SW_SPST, ov-twin:k2-1817UQ, F.Cu at (192.0, 106.0)
- added U6: ~, Package_DFN_QFN:QFN-24-1EP_4x4mm_P0.5mm_EP2.7x2.7mm_ThermalVias, F.Cu at (160.6, 66.8)
- added U7: LIS3DH, Package_LGA:LGA-16_3x3mm_P0.5mm_LayoutBorder3x5y, F.Cu at (172.0, 92.0)
- added U8: SN74LVC1T45DBV, Package_TO_SOT_SMD:SOT-23-6, F.Cu at (190.8, 75.8)
- added Y3: Crystal_GND24, Crystal:Crystal_SMD_3225-4Pin_3.2x2.5mm, F.Cu at (155.8, 67.4)
- moved C13 109.4 mm to (189.6, 64.6), turned to -90 degrees
- moved C14 103.3 mm to (183.8, 69.4)
- moved U1 84.3 mm to (184.0, 64.6), turned to 180 degrees
- moved R3 68.5 mm to (164.4, 65.8)
- moved R4 64.6 mm to (164.4, 64.8)
- moved C22 12.2 mm to (179.4, 79.8), turned to -90 degrees
- moved C26 12.0 mm to (189.4, 83.6)
- moved C1 11.4 mm to (169.4, 78.6)
- moved C10 11.4 mm to (166.4, 77.1)
- moved C11 11.4 mm to (163.4, 77.1)
- moved C12 11.4 mm to (165.8, 88.6)
- moved C15 11.4 mm to (159.0, 90.6)
- moved C16 11.4 mm to (163.8, 90.6)
- moved C17 11.4 mm to (179.0, 90.6)
- moved C18 11.4 mm to (159.8, 71.1), turned to 180 degrees
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Connections:
- J1 pad A4: VBUS -> +5V
- J1 pad A9: VBUS -> +5V
- J1 pad B4: VBUS -> +5V
- J1 pad B9: VBUS -> +5V
- R3 pad 1: unconnected-(R3-Pad1) -> GND
- R4 pad 1: unconnected-(R4-Pad1) -> GND
- U2 pad 4: unconnected-(U2-GPIO2-Pad4) -> /pi-b-swclk
- U2 pad 5: unconnected-(U2-GPIO3-Pad5) -> /pi-b-swdio
- U2 pad 6: unconnected-(U2-GPIO4-Pad6) -> /pi-a-tx-pi-b-rx
- U2 pad 7: unconnected-(U2-GPIO5-Pad7) -> /pi-a-rx-pi-b-tx
- U3 pad 11: unconnected-(U3-GPIO8-Pad11) -> /lis3dh-sdi-sda
- U3 pad 12: unconnected-(U3-GPIO9-Pad12) -> /lis3dh-scl-spc
- U3 pad 13: unconnected-(U3-GPIO10-Pad13) -> /lis3dh-int2
- U3 pad 14: unconnected-(U3-GPIO11-Pad14) -> /lis3dh-int1
- U3 pad 2: unconnected-(U3-GPIO0-Pad2) -> /pi-b-sw-1
- U3 pad 27: unconnected-(U3-GPIO16-Pad27) -> /pi-a-rx-pi-b-tx
- U3 pad 28: unconnected-(U3-GPIO17-Pad28) -> /pi-a-tx-pi-b-rx
- U3 pad 29: unconnected-(U3-GPIO18-Pad29) -> /pi-b-sw-5
- U3 pad 3: unconnected-(U3-GPIO1-Pad3) -> /pi-b-sw-2
- U3 pad 30: unconnected-(U3-GPIO19-Pad30) -> /pi-b-sw-6
- U3 pad 31: unconnected-(U3-GPIO20-Pad31) -> /pi-b-sw-7
- U3 pad 32: unconnected-(U3-GPIO21-Pad32) -> /pi-b-sw-8
- U3 pad 37: unconnected-(U3-GPIO25-Pad37) -> /smartled-3v3
- U3 pad 38: unconnected-(U3-GPIO26_ADC0-Pad38) -> /pi-b-pot
- U3 pad 4: unconnected-(U3-GPIO2-Pad4) -> /pi-b-sw-3
- U3 pad 5: unconnected-(U3-GPIO3-Pad5) -> /pi-b-sw-4
- U3 pad 6: unconnected-(U3-GPIO4-Pad6) -> /lis3dh-sdo-sa0
- U3 pad 7: unconnected-(U3-GPIO5-Pad7) -> /lis3dh-cs
- U3 pad 8: unconnected-(U3-GPIO6-Pad8) -> /lis3dh-scl-spc
- U3 pad 9: unconnected-(U3-GPIO7-Pad9) -> /lis3dh-sdi-sda
Routing:
- net +5V: track 0.00 -> 305.3 mm, vias 0 -> 11
- net +3V3: track 21.4 -> 79.3 mm, vias 4 -> 33
- net /pi-b-sw-2: track 0.00 -> 46.3 mm, vias 0 -> 2
- net /pi-b-sw-4: track 0.00 -> 43.8 mm, vias 0 -> 2
- net /pi-b-pot: track 0.00 -> 41.3 mm, vias 0 -> 1
- net /pi-b-sw-1: track 0.00 -> 38.8 mm, vias 0 -> 2
- net Net-(D8-DOUT): track 0.00 -> 35.6 mm, vias 0 -> 3
- net /pi-b-sw-3: track 0.00 -> 35.4 mm, vias 0 -> 2
- net +1V1: track 13.4 -> 47.6 mm, vias 4 -> 6
- net /pi-b-usb-dm: track 0.00 -> 30.6 mm, vias 0 -> 2
- net /pi-b-usb-dp: track 0.00 -> 29.0 mm, vias 0 -> 2
- net /pi-b-sw-7: track 0.00 -> 25.8 mm, vias 0 -> 2
- net /pi-b-sw-8: track 0.00 -> 25.3 mm, vias 0 -> 2
- net GND: track 24.6 -> 49.3 mm, vias 14 -> 26
- net /lis3dh-scl-spc: track 0.00 -> 24.5 mm, vias 0 -> 3
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- added copper zone on In2.Cu, net +3V3
- added copper zone on F.Cu, net GND
Other:
- outline, holes or cut-outs redrawn

Commit message: Okay let's try it
Routing:
- net /pi-a-tx-pi-b-rx: track 1.95 -> 42.2 mm, vias 1 -> 2
- net /pi-a-rx-pi-b-tx: track 3.02 -> 42.7 mm, vias 1 -> 2
- net /pi-b-swdio: track 1.50 -> 40.5 mm, vias 1 -> 2
- net /pi-b-swclk: track 1.42 -> 39.8 mm, vias 1 -> 2
Changed lines of the file:
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@@
   (segment (start 191.75 76.9375) (end 191.75 77.95) (width 0.2) (layer "F.Cu") (net 2))
   (segment (start 160.7 72.5) (end 160 73.2) (width 0.2) (layer "F.Cu") (net 2))
-  (segment (start 159.48 83.52) (end 159.6 83.4) (width 0.2) (layer "F.Cu") (net 2))
   (segment (start 164.8 79.7625) (end 164.8 79.230025) (width 0.2) (layer "F.Cu") (net 2))
   (segment (start 184.4 79.7625) (end 184.4 78.8) (width 0.2) (layer "F.Cu") (net 2))
@@
   (segment (start 170.775 90.225) (end 171 90) (width 0.2) (layer "F.Cu") (net 2))
   (segment (start 172.5 90.3) (end 172.8 90) (width 0.2) (layer "F.Cu") (net 2))
+  (segment (start 159.48 84.88) (end 159.6 85) (width 0.2) (layer "F.Cu") (net 2))
   (segment (start 164.8 79.230025) (end 165.230025 78.8) (width 0.2) (layer "F.Cu") (net 2))
   (segment (start 164.4 86.105025) (end 163.894975 85.6) (width 0.2) (layer "F.Cu") (net 2))
@@
   (segment (start 163.894975 85.6) (end 163.8 85.6) (width 0.2) (layer "F.Cu") (net 2))
   (segment (start 184.4 78) (end 184.8 78.4) (width 0.2) (layer "F.Cu") (net 2))
+  (segment (start 159.48 84.2) (end 159.48 84.88) (width 0.2) (layer "F.Cu") (net 2))
   (segment (start 184.8 79.230025) (end 185.230025 78.8) (width 0.2) (layer "F.Cu") (net 2))
   (segment (start 164.4 78) (end 164.8 78.4) (width 0.2) (layer "F.Cu") (net 2))
@@
   (segment (start 160.35 61.85) (end 161.2 61) (width 0.25) (layer "F.Cu") (net 2))
   (segment (start 184.4 77.58) (end 184.4 78) (width 0.2) (layer "F.Cu") (net 2))
-  (segment (start 159.48 84.2) (end 159.48 83.52) (width 0.2) (layer "F.Cu") (net 2))
   (segment (start 180.7 71.1) (end 180.7 72.5) (width 0.2) (layer "F.Cu") (net 2))
   (segment (start 160.35 62.2) (end 160.35 61.85) (width 0.25) (layer "F.Cu") (net 2))
@@
   (via (at 188.2 79.2) (size 0.5) (drill 0.3) (layers "F.Cu" "B.Cu") (free) (net 2))
   (via (at 184.4 65.2) (size 0.5) (drill 0.3) (layers "F.Cu" "B.Cu") (free) (net 2))
-  (via (at 159.6 83.4) (size 0.5) (drill 0.3) (layers "F.Cu" "B.Cu") (net 2))
   (via (at 167.4 79.6) (size 0.5) (drill 0.3) (layers "F.Cu" "B.Cu") (free) (net 2))
   (via (at 160 73.2) (size 0.5) (drill 0.3) (layers "F.Cu" "B.Cu") (net 2))
@@
   (via (at 188.2 80) (size 0.5) (drill 0.3) (layers "F.Cu" "B.Cu") (free) (net 2))
   (via (at 164.8 78.4) (size 0.5) (drill 0.3) (layers "F.Cu" "B.Cu") (net 2))
+  (via (at 159.6 85) (size 0.5) (drill 0.3) (layers "F.Cu" "B.Cu") (net 2))
   (via (at 168 79.2) (size 0.5) (drill 0.3) (layers "F.Cu" "B.Cu") (free) (net 2))
   (via (at 185.5 78.8) (size 0.5) (drill 0.3) (layers "F.Cu" "B.Cu") (net 2))
@@
   (segment (start 164.41 89.72) (end 163.8 89.11) (width 0.2) (layer "F.Cu") (net 6))
   (segment (start 186.8 86.6375) (end 188.2375 86.6375) (width 0.2) (layer "F.Cu") (net 7))
+  (segment (start 157.2 82.6) (end 156.8 83) (width 0.2) (layer "F.Cu") (net 7))
   (segment (start 188.2375 86.6375) (end 188.6 87) (width 0.2) (layer "F.Cu") (net 7))
+  (segment (start 160.7625 82.6) (end 157.2 82.6) (width 0.2) (layer "F.Cu") (net 7))
   (via (at 188.6 87) (size 0.5) (drill 0.3) (layers "F.Cu" "B.Cu") (net 7))
+  (via (at 156.8 83) (size 0.5) (drill 0.3) (layers "F.Cu" "B.Cu") (net 7))
+  (segment (start 178.2 88.2) (end 184.8 88.2) (width 0.2) (layer "In2.Cu") (net 7))
+  (segment (start 156.8 83) (end 161 83) (width 0.2) (layer "In2.Cu") (net 7))
+  (segment (start 186 87) (end 188.6 87) (width 0.2) (layer "In2.Cu") (net 7))
+  (segment (start 162.2 87) (end 177 87) (width 0.2) (layer "In2.Cu") (net 7))
+  (segment (start 161.4 83.4) (end 161.4 86.2) (width 0.2) (layer "In2.Cu") (net 7))
+  (segment (start 177 87) (end 178.2 88.2) (width 0.2) (layer "In2.Cu") (net 7))
+  (segment (start 161.4 86.2) (end 162.2 87) (width 0.2) (layer "In2.Cu") (net 7))
+  (segment (start 184.8 88.2) (end 186 87) (width 0.2) (layer "In2.Cu") (net 7))
+  (segment (start 161 83) (end 161.4 83.4) (width 0.2) (layer "In2.Cu") (net 7))
   (segment (start 165.8 65.8) (end 164.91 65.8) (width 0.2) (layer "F.Cu") (net 8))
   (segment (start 173.1005 65) (end 173.25 65.1495) (width 0.2) (layer "F.Cu") (net 8))
@@
   (segment (start 162.3 74.5) (end 163.3 75.5) (width 0.2) (layer "In1.Cu") (net 28))
   (segment (start 187 87.4) (end 188.2 87.4) (width 0.2) (layer "F.Cu") (net 31))
+  (segment (start 157.6 83) (end 156.8 83.8) (width 0.2) (layer "F.Cu") (net 31))
+  (segment (start 160.7625 83) (end 157.6 83) (width 0.2) (layer "F.Cu") (net 31))
   (segment (start 186.4 86.6375) (end 186.4 87.22206) (width 0.2) (layer "F.Cu") (net 31))
   (segment (start 188.2 87.4) (end 188.6 87.8) (width 0.2) (layer "F.Cu") (net 31))
   (segment (start 186.57794 87.4) (end 187 87.4) (width 0.2) (layer "F.Cu") (net 31))
   (segment (start 186.4 87.22206) (end 186.57794 87.4) (width 0.2) (layer "F.Cu") (net 31))
+  (via (at 156.8 83.8) (size 0.5) (drill 0.3) (layers "F.Cu" "B.Cu") (net 31))
   (via (at 188.6 87.8) (size 0.5) (drill 0.3) (layers "F.Cu" "B.Cu") (net 31))
+  (segment (start 176.8 87.4) (end 178 88.6) (width 0.2) (layer "In2.Cu") (net 31))
+  (segment (start 162 87.4) (end 176.8 87.4) (width 0.2) (layer "In2.Cu") (net 31))
+  (segment (start 161 84.2) (end 161 86.4) (width 0.2) (layer "In2.Cu") (net 31))
+  (segment (start 161 86.4) (end 162 87.4) (width 0.2) (layer "In2.Cu") (net 31))
+  (segment (start 185 88.6) (end 185.8 87.8) (width 0.2) (layer "In2.Cu") (net 31))
+  (segment (start 160.6 83.8) (end 161 84.2) (width 0.2) (layer "In2.Cu") (net 31))
+  (segment (start 178 88.6) (end 185 88.6) (width 0.2) (layer "In2.Cu") (net 31))
+  (segment (start 185.8 87.8) (end 188.6 87.8) (width 0.2) (layer "In2.Cu") (net 31))
+  (segment (start 156.8 83.8) (end 160.6 83.8) (width 0.2) (layer "In2.Cu") (net 31))
   (segment (start 165.2 85.6) (end 165.2 86.6375) (width 0.2) (layer "F.Cu") (net 42))
   (segment (start 165.4 85.4) (end 165.2 85.6) (width 0.2) (layer "F.Cu") (net 42))
@@
   (segment (start 183.55 110.915) (end 183.55 114.472183) (width 0.2) (layer "F.Cu") (net 77))
   (segment (start 183.55 114.472183) (end 180.658094 117.364089) (width 0.2) (layer "F.Cu") (net 77))
+  (segment (start 157.6 81.8) (end 156.8 81) (width 0.2) (layer "F.Cu") (net 82))
   (segment (start 185.2 85.727914) (end 185.2 86.6375) (width 0.2) (layer "F.Cu") (net 82))
+  (segment (start 158.2 81.8) (end 157.6 81.8) (width 0.2) (layer "F.Cu") (net 82))
   (segment (start 185.55922 85.368694) (end 185.2 85.727914) (width 0.2) (layer "F.Cu") (net 82))
+  (segment (start 160.7625 81.8) (end 158.2 81.8) (width 0.2) (layer "F.Cu") (net 82))
+  (via (at 156.8 81) (size 0.5) (drill 0.3) (layers "F.Cu" "B.Cu") (net 82))
   (via (at 185.55922 85.368694) (size 0.5) (drill 0.3) (layers "F.Cu" "B.Cu") (net 82))
+  (segment (start 183.531584 87.4) (end 185.55922 85.372364) (width 0.2) (layer "In2.Cu") (net 82))
+  (segment (start 162.2 82.6) (end 162.2 85.8) (width 0.2) (layer "In2.Cu") (net 82))
+  (segment (start 178.6 87.4) (end 183.531584 87.4) (width 0.2) (layer "In2.Cu") (net 82))
+  (segment (start 185.55922 85.372364) (end 185.55922 85.368694) (width 0.2) (layer "In2.Cu") (net 82))
+  (segment (start 162.6 86.2) (end 177.4 86.2) (width 0.2) (layer "In2.Cu") (net 82))
+  (segment (start 177.4 86.2) (end 178.6 87.4) (width 0.2) (layer "In2.Cu") (net 82))
+  (segment (start 157.2 81.4) (end 161 81.4) (width 0.2) (layer "In2.Cu") (net 82))
+  (segment (start 162.2 85.8) (end 162.6 86.2) (width 0.2) (layer "In2.Cu") (net 82))
+  (segment (start 156.8 81) (end 157.2 81.4) (width 0.2) (layer "In2.Cu") (net 82))
+  (segment (start 161 81.4) (end 162.2 82.6) (width 0.2) (layer "In2.Cu") (net 82))
   (segment (start 186.4 85.7) (end 186.005025 85.7) (width 0.2) (layer "F.Cu") (net 83))
   (segment (start 186.005025 85.7) (end 185.6 86.105025) (width 0.2) (layer "F.Cu") (net 83))
+  (segment (start 157 82.2) (end 156.8 82) (width 0.2) (layer "F.Cu") (net 83))
+  (segment (start 160.7625 82.2) (end 157 82.2) (width 0.2) (layer "F.Cu") (net 83))
   (segment (start 185.6 86.105025) (end 185.6 86.6375) (width 0.2) (layer "F.Cu") (net 83))
   (via (at 186.4 85.7) (size 0.5) (drill 0.3) (layers "F.Cu" "B.Cu") (net 83))
+  (via (at 156.8 82) (size 0.5) (drill 0.3) (layers "F.Cu" "B.Cu") (net 83))
+  (segment (start 177.2 86.6) (end 178.4 87.8) (width 0.2) (layer "In2.Cu") (net 83))
+  (segment (start 178.4 87.8) (end 184.3 87.8) (width 0.2) (layer "In2.Cu") (net 83))
+  (segment (start 157 82) (end 157.2 81.8) (width 0.2) (layer "In2.Cu") (net 83))
+  (segment (start 157.2 81.8) (end 160.8 81.8) (width 0.2) (layer "In2.Cu") (net 83))
+  (segment (start 160.8 81.8) (end 161.8 82.8) (width 0.2) (layer "In2.Cu") (net 83))
+  (segment (start 156.8 82) (end 157 82) (width 0.2) (layer "In2.Cu") (net 83))
+  (segment (start 161.8 86) (end 162.4 86.6) (width 0.2) (layer "In2.Cu") (net 83))
+  (segment (start 184.3 87.8) (end 186.4 85.7) (width 0.2) (layer "In2.Cu") (net 83))
+  (segment (start 161.8 82.8) (end 161.8 86) (width 0.2) (layer "In2.Cu") (net 83))
+  (segment (start 162.4 86.6) (end 177.2 86.6) (width 0.2) (layer "In2.Cu") (net 83))
   (segment (start 180.141906 119.435911) (end 178.127817 121.45) (width 0.2) (layer "F.Cu") (net 84))
   (segment (start 178.127817 121.45) (end 172.915 121.45) (width 0.2) (layer "F.Cu") (net 84))
@@
       )
     )
-  )
-  (zone (net 2) (net_name "+3V3") (layer "In2.Cu") (hatch edge 0.5)
-    (priority 4)
-    (connect_pads (clearance 0.25))
-    (min_thickness 0.25) (filled_areas_thickness no)
-    (fill yes (thermal_gap 0.5) (thermal_bridge_width 0.5))
-    (polygon
-      (pts
-        (xy 152 68)
-        (xy 192 68)
-        (xy 192 92)
-        (xy 152 92)
-      )
-    )
