File: ov-twin.kicad_sch (KiCad schematic)
At the start: 31 parts, among them J1 USB_C_Receptacle_USB2.0, J3 Conn_01x02, U1 NCP1117-3.3_SOT223, U2 RP2040, U4 W25Q128JVS, Y1 Crystal_GND24

Commit message: Hub and stuff
Parts:
- added C17, C19, C33, C34: 27p, Capacitor_SMD:C_0402_1005Metric, symbol Device:C
- added C20, C21, C22, C23, C24, C25, C26, C27, C28, C29, C30, C32: 1u, Capacitor_SMD:C_0402_1005Metric, symbol Device:C_Small
- added C31: 1u, Capacitor_SMD:C_0805_2012Metric, symbol Device:C
- added C35, C36: 10u, Capacitor_SMD:C_0805_2012Metric, symbol Device:C
- added J2: Conn_01x02, Connector_PinHeader_2.54mm:PinHeader_1x02_P2.54mm_Vertical, symbol Connector_Generic:Conn_01x02
- added JP1: SolderJumper_2_Open, Jumper:SolderJumper-2_P1.3mm_Open_TrianglePad1.0x1.5mm, symbol Jumper:SolderJumper_2_Open
- added R11, R13, R15: 1k, Resistor_SMD:R_0402_1005Metric, symbol Device:R
- added R12: DNF, Resistor_SMD:R_0402_1005Metric, symbol Device:R
- added R14: 10k, Resistor_SMD:R_0402_1005Metric, symbol Device:R
- added R7, R8: 27, Resistor_SMD:R_0402_1005Metric, symbol Device:R_Small
- added U3: RP2040, ov-twin:RP2040-QFN-56, symbol ov-twin:RP2040
- added U5: W25Q128JVS, Package_SO:SOIC-8_5.23x5.23mm_P1.27mm, symbol RP2040_minimal-rescue:W25Q128JVS-Memory_Flash
- added U6: ~, Package_DFN_QFN:QFN-24-1EP_4x4mm_P0.5mm_EP2.7x2.7mm_ThermalVias, symbol ov-twin:CH334F
- added Y2, Y3: Crystal_GND24, Crystal:Crystal_SMD_3225-4Pin_3.2x2.5mm, symbol Device:Crystal_GND24
Connections:
- net +1V1: now also C29.2, C30.2, C32.2, U3.23 (DVDD), U3.45 (VREG_VOUT), U3.50 (DVDD)
- net +3V3: now also C20.2, C21.2, C22.2, C23.2, C24.2, C25.2, C26.2, C27.2, C28.2, C31.1, C36.1, R12.1, R14.2, U3.1 (IOVDD), U3.10 (IOVDD), U3.22 (IOVDD), U3.33 (IOVDD), U3.42 (IOVDD), U3.43 (ADC_AVDD), U3.44 (VREG_IN), U3.48 (USB_VDD), U3.49 (IOVDD), U5.8 (VCC), U6.20 (VDD33)
- net +5V: now also C35.1, U6.19 (V5)
- net GND: now also R3.1, R4.1, C17.2, C19.2, C20.1, C21.1, C22.1, C23.1, C24.1, C25.1, C26.1, C27.1, C28.1, C29.1, C30.1, C31.2, C32.1, C33.2, C34.2, C35.2, C36.2, J2.2 (Pin_2), U3.19 (TESTEN), U3.57 (GND), U5.4 (GND), U6.25 (GND), Y2.2, Y2.4, Y3.2, Y3.4
- net USB_D+: now also U6.15 (DPU)
- net USB_D-: now also U6.14 (DMU)
- net pi-a-usb-dm: now also U6.11 (DM1)
- net pi-a-usb-dp: now also U6.12 (DP1)
- net ~{USB_BOOT}: now also J2.1 (Pin_1), R11.2
- new net: R7.1, U3.46 (USB_DM)
- new net: C19.1, R13.2, Y2.3
- new net: R14.1, U3.26 (RUN)
- new net: C34.1, JP1.1 (A), R15.2, Y3.3
- new net: R8.1, U3.47 (USB_DP)
- new net hub-xi: C33.1, U6.4 (XI), Y3.1
- new net hub-xo: JP1.2 (B), R15.1, U6.3 (XO)
- new net pi-b-qspi-sclk: U3.52 (QSPI_SCLK), U5.6 (CLK)
- new net pi-b-qspi-sd0: U3.53 (QSPI_SD0), U5.5 (DI(IO0))
- new net pi-b-qspi-sd1: U3.55 (QSPI_SD1), U5.2 (DO(IO1))
- new net pi-b-qspi-sd2: U3.54 (QSPI_SD2), U5.3 (IO2)
- new net pi-b-qspi-sd3: U3.51 (QSPI_SD3), U5.7 (IO3)
- new net pi-b-qspi-ss: R11.1, R12.2, U3.56 (QSPI_SS), U5.1 (~{CS})
- new net pi-b-swclk: U3.24 (SWCLK)
- new net pi-b-swdio: U3.25 (SWD)
- new net pi-b-usb-dm: R7.2, U6.9 (DM2)
- new net pi-b-usb-dp: R8.2, U6.10 (DP2)
- new net pi-b-xin: C17.1, U3.20 (XIN), Y2.1
- new net pi-b-xout: R13.1, U3.21 (XOUT)

Commit message: Mostly routed, wondering how to do sniffing
Parts:
- added D1, D10, D11, D12, D13, D14, D15, D16, D17, D18, D19, D2, D20, D21, D22, D23, D24, D3, D4, D5, D6, D7, D8, D9: WS2812B, LED_SMD:LED_WS2812B-2020_PLCC4_2.0x2.0mm, symbol LED:WS2812B
- added R16, R17: 27, Resistor_SMD:R_0402_1005Metric, symbol Device:R_Small
- added RV1: R_Potentiometer_MountingPin, Potentiometer_THT:Potentiometer_Alps_RK09K_Single_Vertical, symbol Device:R_Potentiometer_MountingPin
- added SW1, SW2, SW3, SW4, SW5, SW6, SW7, SW8: SW_SPST, ov-twin:k2-1817UQ, symbol Switch:SW_SPST
- added U7: LIS3DH, Package_LGA:LGA-16_3x3mm_P0.5mm_LayoutBorder3x5y, symbol Sensor_Motion:LIS3DH
- added U8: SN74LVC1T45DBV, Package_TO_SOT_SMD:SOT-23-6, symbol Logic_LevelTranslator:SN74LVC1T45DBV
Connections:
- net VBUS is gone; now on net +5V: J1.A4 (VBUS), J1.A9 (VBUS), J1.B4 (VBUS), J1.B9 (VBUS)
- net +3V3: now also RV1.1, U7.1 (VDD_IO), U7.14 (VDD), U8.6 (VCCB)
- net +5V: now also D1.1 (VDD), D10.1 (VDD), D11.1 (VDD), D12.1 (VDD), D13.1 (VDD), D14.1 (VDD), D15.1 (VDD), D16.1 (VDD), D17.1 (VDD), D18.1 (VDD), D19.1 (VDD), D2.1 (VDD), D20.1 (VDD), D21.1 (VDD), D22.1 (VDD), D23.1 (VDD), D24.1 (VDD), D3.1 (VDD), D4.1 (VDD), D5.1 (VDD), D6.1 (VDD), D7.1 (VDD), D8.1 (VDD), D9.1 (VDD), U8.1 (VCCA)
- net GND: now also D1.3 (VSS), D10.3 (VSS), D11.3 (VSS), D12.3 (VSS), D13.3 (VSS), D14.3 (VSS), D15.3 (VSS), D16.3 (VSS), D17.3 (VSS), D18.3 (VSS), D19.3 (VSS), D2.3 (VSS), D20.3 (VSS), D21.3 (VSS), D22.3 (VSS), D23.3 (VSS), D24.3 (VSS), D3.3 (VSS), D4.3 (VSS), D5.3 (VSS), D6.3 (VSS), D7.3 (VSS), D8.3 (VSS), D9.3 (VSS), RV1.3, RV1.MP (MountPin), SW1.2 (B), SW2.2 (B), SW3.2 (B), SW4.2 (B), SW5.2 (B), SW6.2 (B), SW7.2 (B), SW8.2 (B), U7.10 (GND), U7.12 (GND), U7.5 (GND)
- net USB_D+: now also R16.1; no longer U6.15 (DPU)
- net USB_D-: now also R17.1; no longer U6.14 (DMU)
- net pi-a-usb-dm: now also U6.7 (DM3); no longer U6.11 (DM1)
- net pi-a-usb-dp: now also U6.8 (DP3); no longer U6.12 (DP1)
- net pi-b-swclk: now also U2.4 (GPIO2)
- net pi-b-swdio: now also U2.5 (GPIO3)
- net pi-b-usb-dm: now also U6.11 (DM1); no longer U6.9 (DM2)
- net pi-b-usb-dp: now also U6.12 (DP1); no longer U6.10 (DP2)
- net pi-a-tx-pi-b-rx: now reaches U2.6 (GPIO4)
- net pi-a-tx-pi-b-rx: now also U3.28 (GPIO17)
- net pi-a-rx-pi-b-tx: now reaches U2.7 (GPIO5)
- net pi-a-rx-pi-b-tx: now also U3.27 (GPIO16)
- net lis3dh-sdi-sda: now reaches U3.11 (GPIO8)
- net lis3dh-sdi-sda: now also U3.9 (GPIO7), U7.6 (SDA/SDI/SDO)
- net lis3dh-scl-spc: now reaches U3.12 (GPIO9)
- net lis3dh-scl-spc: now also U3.8 (GPIO6), U7.4 (SCL/SPC)
- net lis3dh-int2: now reaches U3.13 (GPIO10)
- net lis3dh-int2: now also U7.9 (INT2)
- net lis3dh-int1: now reaches U3.14 (GPIO11)
- net lis3dh-int1: now also U7.11 (INT1)
- net pi-b-sw-1: now reaches U3.2 (GPIO0)
- net pi-b-sw-1: now also SW1.1 (A)
- net pi-b-sw-5: now reaches U3.29 (GPIO18)
- net pi-b-sw-5: now also SW5.1 (A)
- net pi-b-sw-2: now reaches U3.3 (GPIO1)
- net pi-b-sw-2: now also SW2.1 (A)
- net pi-b-sw-6: now reaches U3.30 (GPIO19)
- net pi-b-sw-6: now also SW6.1 (A)
- net pi-b-sw-7: now reaches U3.31 (GPIO20)
- net pi-b-sw-7: now also SW7.1 (A)
- net pi-b-sw-8: now reaches U3.32 (GPIO21)
- net pi-b-sw-8: now also SW8.1 (A)
- net smartled-3v3: now reaches U3.37 (GPIO25)
- net smartled-3v3: now also U8.4 (B)
- net pi-b-pot: now reaches U3.38 (GPIO26_ADC0)
- net pi-b-pot: now also RV1.2
- net pi-b-sw-3: now reaches U3.4 (GPIO2)
- net pi-b-sw-3: now also SW3.1 (A)
- net pi-b-sw-4: now reaches U3.5 (GPIO3)
- net pi-b-sw-4: now also SW4.1 (A)
- net lis3dh-sdo-sa0: now reaches U3.6 (GPIO4)
- net lis3dh-sdo-sa0: now also U7.7 (SDO/SA0)
- net lis3dh-cs: now reaches U3.7 (GPIO5)
- net lis3dh-cs: now also U7.8 (CS)
- new net: D20.2 (DOUT), D21.4 (DIN)
- new net: D19.2 (DOUT), D20.4 (DIN)
- new net: D10.4 (DIN), D9.2 (DOUT)
- new net: D8.2 (DOUT), D9.4 (DIN)
- new net: D1.2 (DOUT), D2.4 (DIN)
- new net: D11.2 (DOUT), D12.4 (DIN)
- new net: D10.2 (DOUT), D11.4 (DIN)
- new net: D17.2 (DOUT), D18.4 (DIN)
- new net: D16.2 (DOUT), D17.4 (DIN)
- new net: D23.2 (DOUT), D24.4 (DIN)
- new net: D22.2 (DOUT), D23.4 (DIN)
- new net: D21.2 (DOUT), D22.4 (DIN)
- new net: D18.2 (DOUT), D19.4 (DIN)
- new net: D13.2 (DOUT), D14.4 (DIN)
- new net: D12.2 (DOUT), D13.4 (DIN)
- new net: R16.2, U6.15 (DPU)
- new net: D7.2 (DOUT), D8.4 (DIN)
- new net: D6.2 (DOUT), D7.4 (DIN)
- new net: D15.2 (DOUT), D16.4 (DIN)
- new net: D14.2 (DOUT), D15.4 (DIN)
- new net: D4.2 (DOUT), D5.4 (DIN)
- new net: D3.2 (DOUT), D4.4 (DIN)
- new net: R17.2, U6.14 (DMU)
- new net: D5.2 (DOUT), D6.4 (DIN)
- new net: D2.2 (DOUT), D3.4 (DIN)
- new net: U8.2 (GND), U8.5 (DIR)
- new net smartled-5v: U8.3 (A)
- new net smartled-5v0: D1.4 (DIN)

Commit message: Add missing decoupling and such
Parts:
- added C37, C38, C39: 1u, Capacitor_SMD:C_0805_2012Metric, symbol Device:C
- added C40, C41, C42, C43, C44, C45: 10u, Capacitor_SMD:C_0805_2012Metric, symbol Device:C
- added R18, R19, R20: 10k, Resistor_SMD:R_0402_1005Metric, symbol Device:R
Connections:
- net +3V3: now also C37.1, C38.1, R18.1, R19.1, R20.1
- net +5V: now also C39.1, C40.1, C41.1, C42.1, C43.1, C44.1, C45.1
- net GND: now also C37.2, C38.2, C39.2, C40.2, C41.2, C42.2, C43.2, C44.2, C45.2
- net lis3dh-cs: now also U2.14 (GPIO11), R20.2
- net lis3dh-int1: now also U2.28 (GPIO17)
- net lis3dh-int2: now also U2.27 (GPIO16)
- net lis3dh-scl-spc: now also U2.15 (GPIO12), U2.18 (GPIO15), R18.2
- net lis3dh-sdi-sda: now also U2.16 (GPIO13), U2.17 (GPIO14), R19.2
- net lis3dh-sdo-sa0: now also U2.13 (GPIO10)
- net pi-b-pot: now also U2.38 (GPIO26_ADC0)
- net pi-b-sw-1: now also U2.29 (GPIO18)
- net pi-b-sw-2: now also U2.30 (GPIO19)
- net pi-b-sw-3: now also U2.31 (GPIO20)
- net pi-b-sw-4: now also U2.32 (GPIO21)
- net pi-b-sw-5: now also U2.34 (GPIO22)
- net pi-b-sw-6: now also U2.35 (GPIO23)
- net pi-b-sw-7: now also U2.36 (GPIO24)
- net pi-b-sw-8: now also U2.37 (GPIO25)
- net smartled-3v3: now also U2.12 (GPIO9)

Commit message: That worked pretty well I thought!
Parts:
- removed C37, C38, C39: 1u, Capacitor_SMD:C_0805_2012Metric, symbol Device:C
- added C37, C38, C39: 1u, Capacitor_SMD:C_0402_1005Metric, symbol Device:C_Small
Connections:
- net smartled-5v is gone; now on net smartled-5v0: U8.3 (A)
- net +3V3: now also C37.2, C38.2
- net +5V: now also C39.2
- net GND: now also U8.2 (GND), U8.5 (DIR), C37.1, C38.1, C39.1
- net lis3dh-int1: now also U2.11 (GPIO8); no longer U2.28 (GPIO17)
- net lis3dh-int2: now also U2.9 (GPIO7); no longer U2.27 (GPIO16)
- net lis3dh-scl-spc: no longer U2.18 (GPIO15)
- net lis3dh-sdi-sda: no longer U2.17 (GPIO14)
- net pi-b-sw-1: now also U2.32 (GPIO21); no longer U2.29 (GPIO18)
- net pi-b-sw-2: now also U2.31 (GPIO20); no longer U2.30 (GPIO19)
- net pi-b-sw-3: now also U2.30 (GPIO19); no longer U2.31 (GPIO20)
- net pi-b-sw-4: now also U2.29 (GPIO18); no longer U2.32 (GPIO21)

Commit message: Updates
Parts:
- removed D1, D10, D11, D12, D13, D14, D15, D16, D17, D18, D19, D2, D20, D21, D22, D23, D24, D3, D4, D5, D6, D7, D8, D9: WS2812B, LED_SMD:LED_WS2812B-2020_PLCC4_2.0x2.0mm, symbol LED:WS2812B
- removed JP1: SolderJumper_2_Open, Jumper:SolderJumper-2_P1.3mm_Open_TrianglePad1.0x1.5mm, symbol Jumper:SolderJumper_2_Open
- removed R16, R17: 27, Resistor_SMD:R_0402_1005Metric, symbol Device:R_Small
- added D1, D10, D11, D12, D13, D14, D15, D16, D17, D18, D19, D2, D20, D21, D22, D23, D24, D3, D4, D5, D6, D7, D8, D9: ~, LED_SMD:LED_WS2812B-2020_PLCC4_2.0x2.0mm, symbol ov-twin:tcwin-tx1812z5
- added D25: LED3, LED_SMD:LED_0603_1608Metric, symbol Device:LED
- added D26: LED1, LED_SMD:LED_0603_1608Metric, symbol Device:LED
- added D27: LEDActive, LED_SMD:LED_0603_1608Metric, symbol Device:LED
- added J4: Conn_01x02, Connector_PinHeader_2.54mm:PinHeader_1x02_P2.54mm_Vertical, symbol Connector_Generic:Conn_01x02
- added R21, R22: 220, Resistor_SMD:R_0402_1005Metric, symbol Device:R
- added R23: 470, Resistor_SMD:R_0402_1005Metric, symbol Device:R
- added TP2, TP4: TestPoint, TestPoint:TestPoint_Pad_D1.5mm, symbol Connector:TestPoint
- C15, C16, C17, C19, C33, C34: value 27p -> 30pf; footprint Capacitor_SMD:C_0402_1005Metric -> Capacitor_SMD:C_0603_1608Metric
Connections:
- net +3V3: now also U6.19 (V5), D27.2 (A), J4.1 (Pin_1)
- net +5V: now also J2.1 (Pin_1), D1.2 (VDD), D10.2 (VDD), D11.2 (VDD), D12.2 (VDD), D13.2 (VDD), D14.2 (VDD), D15.2 (VDD), D16.2 (VDD), D17.2 (VDD), D18.2 (VDD), D19.2 (VDD), D2.2 (VDD), D20.2 (VDD), D21.2 (VDD), D22.2 (VDD), D23.2 (VDD), D24.2 (VDD), D3.2 (VDD), D4.2 (VDD), D5.2 (VDD), D6.2 (VDD), D7.2 (VDD), D8.2 (VDD), D9.2 (VDD); no longer U6.19 (V5)
- net GND: now also C15.1, C16.1, C17.1, C19.1, C33.1, C34.1, D1.4 (VSS), D10.4 (VSS), D11.4 (VSS), D12.4 (VSS), D13.4 (VSS), D14.4 (VSS), D15.4 (VSS), D16.4 (VSS), D17.4 (VSS), D18.4 (VSS), D19.4 (VSS), D2.4 (VSS), D20.4 (VSS), D21.4 (VSS), D22.4 (VSS), D23.4 (VSS), D24.4 (VSS), D3.4 (VSS), D4.4 (VSS), D5.4 (VSS), D6.4 (VSS), D7.4 (VSS), D8.4 (VSS), D9.4 (VSS), J4.2 (Pin_2); no longer C15.2, C16.2, C17.2, C19.2, C33.2, C34.2
- net USB_D+: now also U6.15 (DPU)
- net USB_D-: now also U6.14 (DMU)
- net hub-xi: now also C33.2; no longer C33.1
- net pi-a-xin: now also C15.2; no longer C15.1
- net pi-b-xin: now also C17.2; no longer C17.1
- net smartled-5v0: now also D1.1 (DIN)
- net at R13.2, Y2.3: now also C19.2; no longer C19.1
- net at R5.2, Y1.3: now also C16.2; no longer C16.1
- net at R15.2, Y3.3: now also C34.2; no longer C34.1
- net usb-led3: now reaches U6.13 (LED3/SCL)
- net at U6.18 (PSELF): now also TP4.1
- net usb-led4: now reaches U6.21 (LED4/SDA)
- net usb-led4: now also D25.1 (K), D26.1 (K), R23.2
- net usb-led1: now reaches U6.22 (LED1)
- net usb-led1: now also R21.2
- net usb-led2: now reaches U6.23 (LED2)
- net usb-led2: now also R22.2
- net ~{USB_BOOT} renamed ~{USB_BOOT_A}
- net ~{USB_BOOT_A}: no longer J2.1 (Pin_1), R11.2
- new net: D12.3 (DOUT), D13.1 (DIN)
- new net: D13.3 (DOUT), D14.1 (DIN)
- new net: D25.2 (A), R21.1
- new net: D10.3 (DOUT), D11.1 (DIN)
- new net: D11.3 (DOUT), D12.1 (DIN)
- new net: D7.3 (DOUT), D8.1 (DIN)
- new net: D8.3 (DOUT), D9.1 (DIN)
- new net: D5.3 (DOUT), D6.1 (DIN)
- new net: D6.3 (DOUT), D7.1 (DIN)
- new net: D22.3 (DOUT), D23.1 (DIN)
- new net: D23.3 (DOUT), D24.1 (DIN)
- new net: D14.3 (DOUT), D15.1 (DIN)
- new net: D26.2 (A), R22.1
- new net: D18.3 (DOUT), D19.1 (DIN)
- new net: D19.3 (DOUT), D20.1 (DIN)
- new net: D1.3 (DOUT), D2.1 (DIN)
- new net: D2.3 (DOUT), D3.1 (DIN)
- new net: D10.1 (DIN), D9.3 (DOUT)
- new net: D3.3 (DOUT), D4.1 (DIN)
- new net: D16.3 (DOUT), D17.1 (DIN)
- new net: D17.3 (DOUT), D18.1 (DIN)
- new net: D4.3 (DOUT), D5.1 (DIN)
- new net: D20.3 (DOUT), D21.1 (DIN)
- new net: D21.3 (DOUT), D22.1 (DIN)
- new net: D15.3 (DOUT), D16.1 (DIN)
- new net: D27.1 (K), R23.1
- new net ~{USB_BOOT_B}: R11.2, TP2.1
- no-connect marks 2 -> 9

Commit message: Second order
Parts:
- removed C33, C34: 30pf, Capacitor_SMD:C_0603_1608Metric, symbol Device:C
- removed R15: 1k, Resistor_SMD:R_0402_1005Metric, symbol Device:R
- added T1, T2: ~, ov-twin:tooling-hole, symbol ov-twin:tooling-hole
- added TP1, TP3: TestPoint, TestPoint:TestPoint_Pad_D1.5mm, symbol Connector:TestPoint
Connections:
- net GND: now also TP3.1
- net hub-xo: now also Y3.3
- net at R14.1, U3.26 (RUN): now also TP1.1
Other:
- moved on the sheet: R14

Commit message: Plot schematic (and clean up schematic a bit)
Other:
- note added: "02"
- note added: "3v3 to 5v0 Level Shifter"
- note added: "5v0 to 3v3 LDO Regulator"
- note added: "Accelerometer LIS3DH"
- note added: "Analog Potentiometer"
- note added: "Assembly Tooling Holes"
- note added: "Debug Microcontroller"
- note added: "OneVariable Twin Trainer"
- note added: "Power Headers"
- note added: "SmartLEDs"
- note added: "Target Microcontroller"
- note added: "Thumb Buttons"
- note added: "USB Hub CH334F"
- note added: "USB-C Socket"
- moved on the sheet: C13, C14, C35, C36, C38, C39, C40, C41, C42, C43, C44, C45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
